File: pico3/pico3.kicad_sch (KiCad schematic)
At the start: 0 parts

Commit message: prueba 3 para mejorar
Parts:
- added U1: RP2040, Package_DFN_QFN:QFN-56-1EP_7x7mm_P0.4mm_EP3.2x3.2mm, symbol MCU_RaspberryPi:RP2040
Connections:
- new net: U1.1 (IOVDD), U1.10 (IOVDD), U1.22 (IOVDD), U1.33 (IOVDD), U1.42 (IOVDD), U1.49 (IOVDD)
- new net: U1.23 (DVDD), U1.50 (DVDD)
Changed lines of the file:
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@@
 	(generator_version "9.0")
 	(paper "A4")
+	(symbol
+		(lib_id "MCU_RaspberryPi:RP2040")
+		(at 181.61 77.47 0)
+		(unit 1)
+		(exclude_from_sim no)
+		(in_bom yes)
+		(on_board yes)
+		(dnp no)
+		(fields_autoplaced yes)
+		(property "Reference" "U1"
+			(at 183.7533 121.92 0)
+			(effects
+				(font
+					(size 1.27 1.27)
+				)
+				(justify left)
+			)
+		)
+		(property "Value" "RP2040"
+			(at 183.7533 124.46 0)
+			(effects
+				(font
+					(size 1.27 1.27)
+				)
+				(justify left)
+			)
+		)
+		(property "Footprint" "Package_DFN_QFN:QFN-56-1EP_7x7mm_P0.4mm_EP3.2x3.2mm"
+			(at 181.61 77.47 0)
+			(effects
+				(font
+					(size 1.27 1.27)
+				)
+				(hide yes)
+			)
+		)
+		(property "Datasheet" "https://datasheets.raspberrypi.com/rp2040/rp2040-datasheet.pdf"
+			(at 181.61 77.47 0)
+			(effects
+				(font
+					(size 1.27 1.27)
+				)
+				(hide yes)
+			)
+		)
+		(property "Description" "A microcontroller by Raspberry Pi"
+			(at 181.61 77.47 0)
+			(effects
+				(font
+					(size 1.27 1.27)
+				)
+				(hide yes)
+			)
+		)
+		(pin "12"
+		)
+		(pin "56"
+		)
+		(pin "24"
+		)
+		(pin "8"
+		)
+		(pin "28"
+		)
+		(pin "31"
+		)
+		(pin "35"
+		)
+		(pin "38"
+		)
+		(pin "29"
+		)
+		(pin "33"
+		)
+		(pin "37"
+		)
+		(pin "22"
+		)
+		(pin "48"
+		)
+		(pin "19"
+		)
+		(pin "9"
+		)
+		(pin "54"
+		)
+		(pin "52"
+		)
+		(pin "6"
+		)
+		(pin "7"
+		)
+		(pin "34"
+		)
+		(pin "25"
+		)
+		(pin "42"
+		)
+		(pin "26"
+		)
+		(pin "44"
+		)
+		(pin "13"
+		)
+		(pin "55"
+		)
+		(pin "15"
+		)
+		(pin "51"
+		)
+		(pin "16"
+		)
+		(pin "23"
+		)
+		(pin "10"
+		)
+		(pin "3"
+		)
+		(pin "45"
+		)
+		(pin "4"
+		)
+		(pin "57"
+		)
+		(pin "47"
+		)
+		(pin "53"
+		)
+		(pin "21"
+		)
+		(pin "46"
+		)
+		(pin "20"
+		)
+		(pin "50"
+		)
+		(pin "1"
+		)
+		(pin "49"
+		)
+		(pin "43"
+		)
+		(pin "2"
+		)
+		(pin "5"
+		)
+		(pin "11"
+		)
+		(pin "14"
+		)
+		(pin "17"
+		)
+		(pin "18"
+		)
+		(pin "27"
+		)
+		(pin "30"
+		)
+		(pin "32"
+		)
+		(pin "36"
+		)
+		(pin "39"
+		)
+		(pin "40"
+		)
+		(pin "41"
+		)
+		(instances
+			(project ""
+				(path "/1a09daab-4624-438a-a005-d7b95b96fc64"
+					(reference "U1")
+					(unit 1)
+				)
+			)
+		)
+	)
 	(sheet_instances
 		(path "/"

Commit message: son muchas pruebas, pero parece que ya le estoy entendiendo
Connections:
- net at U1.28 (GPIO17): now also U1.53 (QSPI_SD0)
Changed lines of the file:
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@@
 	(generator_version "9.0")
 	(paper "A4")
+	(wire
+		(pts
+			(xy 135.89 62.23) (xy 135.89 29.21)
+		)
+		(stroke
+			(width 0)
+			(type default)
+		)
+	)
+	(wire
+		(pts
+			(xy 215.9 29.21) (xy 215.9 82.55)
+		)
+		(stroke
+			(width 0)
+			(type default)
+		)
+	)
+	(wire
+		(pts
+			(xy 135.89 29.21) (xy 215.9 29.21)
+		)
+		(stroke
+			(width 0)
+			(type default)
+		)
+	)
+	(wire
+		(pts
+			(xy 156.21 62.23) (xy 135.89 62.23)
+		)
+		(stroke
+			(width 0)
+			(type default)
+		)
+	)
+	(wire
+		(pts
+			(xy 215.9 82.55) (xy 207.01 82.55)
+		)
+		(stroke
+			(width 0)
+			(type default)
+		)
+	)
 	(symbol
 		(lib_id "MCU_RaspberryPi:RP2040")
